File: LrtraPCB.kicad_pcb (KiCad board)
At the start: 2 copper layers, 90 x 54 mm, 28 parts, among them SW1 SW_DPDT_x2, U1 LMC555CM/NOPB

Commit message: [modify] modify sign
Parts:
- removed david11014: CC-BY-NC-SA, Img:CC-BY-NC-SA
- added LutraRescutePCBBusinessCard: CC-BY-NC-SA, Img:CC-BY-NC-SA, B.Cu at (185.3, 96.9)
